File: Reservoir_Circuit.kicad_pcb (KiCad board)
At the start: 2 copper layers, 70 x 57.5 mm, 27 parts, among them J1 CN7, J2 CN10, J3 ECE298_RS_PWR_EXT, M1 Motor_Servo, M2 Motor_DC, U1 CD74HC540E, U2 HC-SR04, U5 L9110S

Commit message: Added potentiometer and test points; clean ERC results
Parts:
- added C10: 100pF, Capacitor_SMD:C_1206_3216Metric, B.Cu at (156.5, 77.0)
- added C9: 10nF, Capacitor_SMD:C_1206_3216Metric, B.Cu at (156.5, 72.0)
- added RV1: R_Potentiometer_US, Potentiometer_SMD:Potentiometer_Bourns_3314J_Vertical, F.Cu at (117.5, 86.0)
- added TP2: TP_POT, Connector_PinHeader_1.00mm:PinHeader_1x01_P1.00mm_Vertical, F.Cu at (115.0, 98.5)
- added TP3: TP_SERVO, Connector_PinHeader_1.00mm:PinHeader_1x01_P1.00mm_Vertical, F.Cu at (155.5, 89.0)
- added TP4: TP_RPM, Connector_PinHeader_1.00mm:PinHeader_1x01_P1.00mm_Vertical, F.Cu at (154.0, 83.0)
- added U6: ~, Connector_PinHeader_2.54mm:PinHeader_1x04_P2.54mm_Vertical, F.Cu at (152.3, 70.8)
- moved M1 0.51 mm to (159.0, 109.0)
Connections:
- J1 pad 19: GND -> unconnected-(J1-Pin_19-Pad19)
- J1 pad 22: GND -> unconnected-(J1-Pin_22-Pad22)
- J1 pad 38: unconnected-(J1-Pin_38-Pad38) -> /PC0
- J2 pad 20: GND -> unconnected-(J2-Pin_20-Pad20)
- J2 pad 22: unconnected-(J2-Pin_22-Pad22) -> /PB2
- J2 pad 32: GND -> unconnected-(J2-Pin_32-Pad32)
Routing:
- net GND: track 231.3 -> 314.8 mm, vias 5 -> 9
- net +3V3: track 67.6 -> 133.0 mm, vias 1 -> 6
- net /PC0: track 0.00 -> 31.1 mm, vias 0 -> 2
- net /PB2: track 0.00 -> 27.3 mm, vias 0 -> 1
- net /SERVO_SIG: track 17.7 -> 32.8 mm, vias 1 -> 2
- net /PB5: track 56.5 -> 44.6 mm
- net /G_BUF: track 8.46 -> 13.3 mm
- net /PB8: track 55.2 -> 59.6 mm
- net /PB9: track 55.3 -> 59.4 mm
- net /PC9: track 61.1 -> 63.8 mm
- net /PB6: track 44.3 -> 41.7 mm
- net /PA11: track 23.3 -> 25.6 mm
- net /PA8: track 8.61 -> 10.0 mm
- net /PA1: track 38.8 -> 38.0 mm
- net /PC8: track 69.9 -> 70.7 mm
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